File: hardware/chufebu-v-0-rev-a/chufebu-v-0-rev-a.kicad_sch (KiCad schematic)
At the start: 12 parts, among them J1 Conn_02x08_Odd_Even, J10 Conn_01x04_Pin, J2 Conn_02x08_Odd_Even, J3 Conn_02x08_Odd_Even, J4 Conn_01x04_Pin, J5 Conn_01x04_Pin, J6 Conn_01x04_Pin, J7 Conn_02x08_Odd_Even, J8 Conn_02x08_Odd_Even, J9 Conn_01x04_Pin

Commit message: agregar documentacion
Other:
- title: chufebu-v-0 -> chufebu v0.1
Changed lines of the file:
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@@
 	(paper "A5")
 	(title_block
-		(title "chufebu-v-0")
+		(title "chufebu v0.1")
 		(date "2026-10-02")
 		(rev "rev-a")
